Commit message: Add the peg end effector to the robot description
A fixed peg link on the flange face with its axis along link6 z, and a peg_tcp
frame 60 mm out at the tip, which is the frame the kinematics solve for. No
inertial element: the peg's mass is not known, so the dynamics are unchanged.

hole.stl is the mating part, tracked as an asset but not yet wired into any
scene.

File: workspace/src/agx_reference/piper/piper/urdf/piper_description.urdf (robot description, URDF)
Before this commit: robot piper, 8 links, 7 joints
Links:
- added link peg; collision mesh filename=meshes/peg.stl scale=0.001 0.001 0.001; visual mesh filename=meshes/peg.stl scale=0.001 0.001 0.001
- added link peg_tcp
Joints:
- added joint link6_to_peg: type fixed, parent link6, child peg, origin xyz=0 0 0 rpy=0 0 0
- added joint peg_to_peg_tcp: type fixed, parent peg, child peg_tcp, origin xyz=0 0 0.06 rpy=0 0 0
